File: project/LEMCurrentSensor/LEMCurrentSensor.kicad_pcb (KiCad board)
At the start: 2 copper layers, 40 x 40 mm, 18 parts, among them J1 Conn_01x01_Female, J2 Conn_01x01_Female, J3 Conn_01x03_Female, U1 LTSR25-NP, U2 AD8651

Commit message: 発注用データ作成
Parts:
- moved TP3 2.69 mm to (98.0, 49.0)
Routing:
- net GND: track 12.2 -> 14.3 mm
Other:
- board text added: "+"
- board text added: "-"
- board text added: "1"
- board text added: "3"
- board text added: "5V"
- board text added: "CS"
- board text added: "Current sensor ver1.0-LEM"
- board text added: "GND"
- board text added: "Vout"
Changed lines of the file:
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@@
   (general
     (thickness 1.6)
-    (drawings 6)
+    (drawings 16)
     (tracks 55)
     (zones 0)
@@
     (descr "LEM current transducer LEM_LTSR-NP 5V supply voltage series https://www.lem.com/sites/default/files/products_datasheets/ltsr_6-np.pdf")
     (tags "Current transducer")
-    (fp_text reference U1 (at -5 0 180) (layer F.SilkS)
+    (fp_text reference U1 (at -5.6 -0.2 180) (layer F.SilkS)
       (effects (font (size 1 1) (thickness 0.15)))
     )
@@
     (tags "capacitor handsolder")
     (attr smd)
-    (fp_text reference C1 (at 0 -1.43) (layer F.SilkS)
+    (fp_text reference C1 (at -0.0375 1.55) (layer F.SilkS)
       (effects (font (size 1 1) (thickness 0.15)))
     )
@@
     (tags "capacitor handsolder")
     (attr smd)
-    (fp_text reference C2 (at 0 -1.43 270) (layer F.SilkS)
+    (fp_text reference C2 (at 2.6625 0 270) (layer F.SilkS)
       (effects (font (size 1 1) (thickness 0.15)))
     )
@@
     (tags "capacitor handsolder")
     (attr smd)
-    (fp_text reference C3 (at 0 -1.43) (layer F.SilkS)
+    (fp_text reference C3 (at 2.6625 0) (layer F.SilkS)
       (effects (font (size 1 1) (thickness 0.15)))
     )
@@
     (tags "test point SMD pad rectangle square")
     (attr virtual)
-    (fp_text reference J2 (at 0 -2.898) (layer F.SilkS)
+    (fp_text reference J2 (at 0 -2.898) (layer F.SilkS) hide
       (effects (font (size 1 1) (thickness 0.15)))
     )
@@
     (tags "resistor handsolder")
     (attr smd)
-    (fp_text reference R1 (at 0 -1.43 180) (layer F.SilkS)
+    (fp_text reference R1 (at -2.7125 0.1 180) (layer F.SilkS)
       (effects (font (size 1 1) (thickness 0.15)))
     )
@@
     (tags "resistor handsolder")
     (attr smd)
-    (fp_text reference R2 (at 0 -1.43) (layer F.SilkS)
+    (fp_text reference R2 (at 2.7125 0) (layer F.SilkS)
       (effects (font (size 1 1) (thickness 0.15)))
     )
@@
     (tags "resistor handsolder")
     (attr smd)
-    (fp_text reference R3 (at 0 -1.43 180) (layer F.SilkS)
+    (fp_text reference R3 (at 2.4125 1 180) (layer F.SilkS)
       (effects (font (size 1 1) (thickness 0.15)))
     )
@@
     (descr "solder Pin_ with flat fork, hole diameter 0.7mm, length 6.5mm, width 1.8mm")
     (tags "solder Pin_ with flat fork")
-    (fp_text reference TP1 (at 0 1.8) (layer F.SilkS)
+    (fp_text reference TP1 (at 0 2.2) (layer F.SilkS)
       (effects (font (size 1 1) (thickness 0.15)))
     )
@@
     (descr "solder Pin_ with flat fork, hole diameter 0.7mm, length 6.5mm, width 1.8mm")
     (tags "solder Pin_ with flat fork")
-    (fp_text reference TP2 (at 0 1.8) (layer F.SilkS)
+    (fp_text reference TP2 (at 0 -2) (layer F.SilkS)
       (effects (font (size 1 1) (thickness 0.15)))
     )
@@
     (tags "test point SMD pad rectangle square")
     (attr virtual)
-    (fp_text reference J1 (at 0 -2.898) (layer F.SilkS)
+    (fp_text reference J1 (at 0 -2.898) (layer F.SilkS) hide
       (effects (font (size 1 1) (thickness 0.15)))
     )
@@
     (tags "mounting hole 3.2mm no annular m3")
     (attr virtual)
-    (fp_text reference H1 (at 0 -4.2) (layer F.SilkS)
+    (fp_text reference H1 (at 0 -4.2) (layer F.SilkS) hide
       (effects (font (size 1 1) (thickness 0.15)))
     )
@@
     (tags "mounting hole 3.2mm no annular m3")
     (attr virtual)
-    (fp_text reference H2 (at 0 -4.2) (layer F.SilkS)
+    (fp_text reference H2 (at 0 -4.2) (layer F.SilkS) hide
       (effects (font (size 1 1) (thickness 0.15)))
     )
@@
     (tags "mounting hole 3.2mm no annular m3")
     (attr virtual)
-    (fp_text reference H3 (at 0 -4.2) (layer F.SilkS)
+    (fp_text reference H3 (at 0 -4.2) (layer F.SilkS) hide
       (effects (font (size 1 1) (thickness 0.15)))
     )
@@
     (tags "mounting hole 3.2mm no annular m3")
     (attr virtual)
-    (fp_text reference H4 (at 0 -4.2) (layer F.SilkS)
+    (fp_text reference H4 (at 0 -4.2) (layer F.SilkS) hide
       (effects (font (size 1 1) (thickness 0.15)))
     )
@@
   )
   (module Connector_Pin:Pin_D0.7mm_L6.5mm_W1.8mm_FlatFork (layer F.Cu)
-    (at 100.5 48)
+    (at 98 49)
     (descr "solder Pin_ with flat fork, hole diameter 0.7mm, length 6.5mm, width 1.8mm")
     (tags "solder Pin_ with flat fork")
-    (fp_text reference TP3 (at 0 1.8) (layer F.SilkS)
+    (fp_text reference TP3 (at 0 2.4) (layer F.SilkS)
       (effects (font (size 1 1) (thickness 0.15)))
     )
@@
     )
   )
+  (gr_text "Current sensor ver1.0-LEM\n" (at 84.9 57.9) (layer B.SilkS)
+    (effects (font (size 1.3 1.3) (thickness 0.3)) (justify mirror))
+  )
+  (gr_text Vout (at 88.6 50.2) (layer F.SilkS)
+    (effects (font (size 1.5 1.5) (thickness 0.2)))
+  )
+  (gr_text 3 (at 101 43.5) (layer F.SilkS)
+    (effects (font (size 1 1) (thickness 0.1)))
+  )
+  (gr_text 1 (at 101.5 38) (layer F.SilkS)
+    (effects (font (size 1 1) (thickness 0.1)))
+  )
+  (gr_text CS (at 103 47) (layer F.SilkS)
+    (effects (font (size 1.5 1.5) (thickness 0.2)))
+  )
+  (gr_text GND (at 102.5 49) (layer F.SilkS)
+    (effects (font (size 1.5 1.5) (thickness 0.2)))
+  )
+  (gr_text 5V (at 103 45) (layer F.SilkS)
+    (effects (font (size 1.5 1.5) (thickness 0.2)))
+  )
+  (gr_text CS (at 97.5 32) (layer F.SilkS)
+    (effects (font (size 1.5 1.5) (thickness 0.2)))
+  )
+  (gr_text - (at 71 49.5) (layer F.SilkS)
+    (effects (font (size 1.5 1.5) (thickness 0.3)))
+  )
+  (gr_text + (at 71 29.5) (layer F.SilkS)
+    (effects (font (size 1.5 1.5) (thickness 0.3)))
+  )
   (gr_line (start 105 60) (end 105 20) (layer Edge.Cuts) (width 0.2))
   (gr_line (start 65 60) (end 105 60) (layer Edge.Cuts) (width 0.2))
@@
   (segment (start 101.32 40.2) (end 98.8 40.2) (width 0.25) (layer F.Cu) (net 1))
   (segment (start 103.2 42.08) (end 101.32 40.2) (width 0.25) (layer F.Cu) (net 1))
-  (segment (start 103.2 45.3) (end 103.2 42.08) (width 0.25) (layer F.Cu) (net 1))
-  (segment (start 100.5 48) (end 103.2 45.3) (width 0.25) (layer F.Cu) (net 1))
+  (segment (start 103.2 43.8) (end 98 49) (width 0.25) (layer F.Cu) (net 1))
+  (segment (start 103.2 42.08) (end 103.2 43.8) (width 0.25) (layer F.Cu) (net 1))
   (segment (start 100.275 37) (end 98.8 38.475) (width 0.25) (layer F.Cu) (net 2))
   (segment (start 103.2 37) (end 100.275 37) (width 0.25) (layer F.Cu) (net 2))
